File: PCB/replica.sch (KiCad schematic (older format))
At the start: 45 parts, among them J1 USB_B, SW1 SW_Push, SW2 SW_Push, U1 W65C02S6TPG-14, U10 74HCT04, U11 74LS138, U12 TXS0108EPW, U2 AT28C64B-15PU, U3 AS6C62256-55PCN, U4 6821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

Commit message: pcb layout
Parts:
- added J2: Conn_01x03, Connector_PinHeader_2.54mm:PinHeader_1x03_P2.54mm_Vertical, symbol Connector_Generic:Conn_01x03
- C1, C10, C11, C12, C13, C14, C15, C16, C19, C2, C3, C4, C5, C7, C8, C9: footprint (none) -> Capacitor_SMD:C_0603_1608Metric; symbol Device:C_Small -> replica-rescue:C_Small-Device
- C17, C18: footprint (none) -> Capacitor_SMD:C_1206_3216Metric; symbol Device:CP1_Small -> replica-rescue:CP1_Small-Device
- C20: renamed from C?; footprint (none) -> Capacitor_SMD:C_0603_1608Metric; symbol Device:C_Small -> replica-rescue:C_Small-Device
- C21: renamed from C7; footprint (none) -> Capacitor_SMD:C_0603_1608Metric; symbol Device:C_Small -> replica-rescue:C_Small-Device
- C22: renamed from C8; footprint (none) -> Capacitor_SMD:C_0603_1608Metric; symbol Device:C_Small -> replica-rescue:C_Small-Device
- C23: renamed from C9; footprint (none) -> Capacitor_SMD:C_0603_1608Metric; symbol Device:C_Small -> replica-rescue:C_Small-Device
- C6: footprint (none) -> Capacitor_SMD:CP_Elec_8x10; symbol Device:CP1_Small -> replica-rescue:CP1_Small-Device
- J1: footprint (none) -> Connector_USB:USB_B_OST_USB-B1HSxx_Horizontal; symbol Connector:USB_B -> replica-rescue:USB_B-Connector
- R1, R2, R3, R4, R5, R6: footprint (none) -> Resistor_SMD:R_0603_1608Metric; symbol Device:R_Small -> replica-rescue:R_Small-Device
- SW1, SW2: footprint (none) -> Button_Switch_SMD:SW_Push_1P1T_NO_6x6mm_H9.5mm; symbol Switch:SW_Push -> replica-rescue:SW_Push-Switch
- U1: footprint DIP1524W56P254L5207H508Q40N -> Package_DIP:DIP-40_W15.24mm
- U10: footprint (none) -> Package_SO:TSSOP-14_4.4x5mm_P0.65mm; symbol 74xx:74HCT04 -> replica-rescue:74HCT04-74xx
- U11: footprint (none) -> Package_SO:TSSOP-16_4.4x5mm_P0.65mm; symbol 74xx:74LS138 -> replica-rescue:74LS138-74xx
- U12, U6, U7: symbol Logic_LevelTranslator:TXS0108EPW -> replica-rescue:TXS0108EPW-Logic_LevelTranslator
- U2: footprint DIP1556W56P254L3702H483Q28N -> Package_DIP:DIP-28_W15.24mm
- U3: footprint DIP1587W140P254L3632H381Q28N -> Package_DIP:DIP-28_W15.24mm
- U4: symbol Interface:6821 -> replica-rescue:6821-Interface
- U5: symbol MCU_ST_STM32F1:STM32F103C8Tx -> replica-rescue:STM32F103C8Tx-MCU_ST_STM32F1
- U8: symbol Regulator_Linear:MIC5219-3.6YM5 -> replica-rescue:MIC5219-3.6YM5-Regulator_Linear
- U9: footprint (none) -> Package_SO:TSSOP-14_4.4x5mm_P0.65mm; symbol 74xx:74HCT00 -> replica-rescue:74HCT00-74xx
- X1: symbol Oscillator:SG-5032CAN -> replica-rescue:SG-5032CAN-Oscillator
